File: techin514-final-project/techin514-final-project.kicad_pcb (KiCad board)
At the start: 2 copper layers, 68.6 x 53.3 mm, 8 parts, among them U1 MOUDLE-SEEEDUINO-XIAO-ESP32C3, U2 HC-SR04, U3 MPU-6050

Commit message: Add sensor code
Parts:
- removed C1, C2: 0.1 mF, Capacitor_SMD:CP_Elec_3x5.3
- removed C3: 2.2 nF, Capacitor_SMD:CP_Elec_3x5.3
- removed U2: HC-SR04, 2025_SR04:XCVR_HC-SR04
- removed U3: MPU-6050, 2025_MPU6050:QFN50P400X400X95-24N
- added BT1: Battery_Cell, Connector_JST:JST_PH_B2B-PH-K_1x02_P2.00mm_Vertical, F.Cu at (69.1, 76.2)
- added D1: LED, LED_THT:LED_D5.0mm, F.Cu at (86.4, 66.0)
- added D2: LED, LED_THT:LED_D5.0mm, F.Cu at (104.1, 106.7)
- added J1: Conn_01x02_Pin, Connector_JST:JST_PH_B2B-PH-K_1x02_P2.00mm_Vertical, F.Cu at (89.4, 81.3)
- added M1: Stepper_Motor_bipolar, 2025_X27_168:x27_stepper_two_holes, F.Cu at (124.5, 78.7)
- added SW1: SW_SPDT, Connector_JST:JST_EH_B3B-EH-A_1x03_P2.50mm_Vertical, F.Cu at (73.6, 66.0)
- R1, R2: value 0 -> R; footprint Resistor_SMD:R_0805_2012Metric_Pad1.20x1.40mm_HandSolder -> Resistor_THT:R_Axial_DIN0207_L6.3mm_D2.5mm_P15.24mm_Horizontal
- U1: footprint 2025_XIAO:MOUDLE14P-SMD-2.54-21X17.8MM -> 2025_XIAO:XIAO_ESP32_SENSE
- moved R2 18.5 mm to (86.4, 99.1)
- moved U1 16.0 mm to (73.7, 96.5)
- moved R1 10.9 mm to (81.3, 73.7)
Connections:
- R1 pad 1: Net-(U1-5V) -> Net-(J1-Pin_1)
- R2 pad 1: Net-(U1-5V) -> Net-(U1-PA8_A4_D4_SDA)
- U1 pad 12: unconnected-(U1-3V3-Pad12) -> Net-(J1-Pin_1)
- U1 pad 14: Net-(U1-5V) -> unconnected-(U1-5V-Pad14)
- U1 pad 4: unconnected-(U1-PA11_A3_D3-Pad4) -> Net-(U1-PA11_A3_D3)
- U1 pad 6: Net-(U1-PA9_A5_D5_SCL) -> unconnected-(U1-PA9_A5_D5_SCL-Pad6)
Routing:
- net GND: track 216.0 -> 85.7 mm
- net Net-(J1-Pin_1): track 0.00 -> 86.9 mm, vias 0 -> 2
- net Net-(U1-5V): track 73.4 -> 0.00 mm
- net Net-(U1-PA11_A3_D3): track 0.00 -> 64.4 mm, vias 0 -> 2
- net Net-(U1-PA9_A5_D5_SCL): track 59.4 -> 0.00 mm
- net Net-(U1-PA8_A4_D4_SDA): track 70.9 -> 13.8 mm
- net Net-(U1-PA10_A2_D2): track 68.8 -> 46.6 mm, vias 0 -> 2
- net Net-(U1-PA02_A0_D0): track 82.9 -> 66.1 mm, vias 0 -> 2
- net Net-(U3-CPOUT): track 12.3 -> 0.00 mm
- net Net-(BT1-+): track 0.00 -> 11.5 mm
- net Net-(U3-REGOUT): track 9.36 -> 0.00 mm
- net Net-(M1--): track 79.6 -> 71.2 mm, vias 0 -> 2
- net Net-(D1-A): track 25.1 -> 17.3 mm
- net Net-(D2-A): track 12.2 -> 11.2 mm
Other:
- board text added: "Hazel Chen Display Circuit v2.0"
- board text removed: "Hazel Chen Sensor Circuit v1.0"
